Commit message: Works but doesnt fly

File: models/rotors_description/urdf/component_snippets.xacro (robot description, xacro)
@@ -273,4 +273,72 @@
             <zero_position_armed>0</zero_position_armed>
             <joint_control_type>position</joint_control_type>
+          </channel>
+        </control_channels>
+      </plugin>
+    </gazebo>
+  </xacro:macro>
+  <!-- Macro to add the mavlink interface. -->
+  <xacro:macro name="mavlink_interface_macro_fw" params="namespace imu_sub_topic gps_sub_topic mag_sub_topic baro_sub_topic mavlink_addr mavlink_udp_port mavlink_tcp_port serial_enabled serial_device baudrate qgc_addr qgc_udp_port sdk_addr sdk_udp_port hil_mode hil_state_level vehicle_is_tailsitter send_vision_estimation send_odometry enable_lockstep use_tcp">
+    <gazebo>
+      <plugin name="mavlink_interface" filename="libgazebo_mavlink_interface.so">
+        <robotNamespace>${namespace}</robotNamespace>
+        <imuSubTopic>${imu_sub_topic}</imuSubTopic>
+        <gpsSubTopic>${gps_sub_topic}</gpsSubTopic>
+        <magSubTopic>${mag_sub_topic}</magSubTopic>
+        <baroSubTopic>${baro_sub_topic}</baroSubTopic>
+        <mavlink_addr>$(arg mavlink_addr)</mavlink_addr>
+        <mavlink_udp_port>$(arg mavlink_udp_port)</mavlink_udp_port>
+        <mavlink_tcp_port>$(arg mavlink_tcp_port)</mavlink_tcp_port>
+        <serialEnabled>$(arg serial_enabled)</serialEnabled>
+        <serialDevice>$(arg serial_device)</serialDevice>
+        <baudRate>$(arg baudrate)</baudRate>
+        <qgc_addr>$(arg qgc_addr)</qgc_addr>
+        <qgc_udp_port>$(arg qgc_udp_port)</qgc_udp_port>
+        <sdk_addr>$(arg sdk_addr)</sdk_addr>
+        <sdk_udp_port>$(arg sdk_udp_port)</sdk_udp_port>
+        <hil_mode>$(arg hil_mode)</hil_mode>
+        <hil_state_level>$(arg hil_state_level)</hil_state_level>
+        <vehicle_is_tailsitter>$(arg vehicle_is_tailsitter)</vehicle_is_tailsitter>
+        <send_vision_estimation>$(arg send_vision_estimation)</send_vision_estimation>
+        <send_odometry>$(arg send_odometry)</send_odometry>
+        <enable_lockstep>$(arg enable_lockstep)</enable_lockstep>
+        <use_tcp>$(arg use_tcp)</use_tcp>
+        <motorSpeedCommandPubTopic>/gazebo/command/motor_speed</motorSpeedCommandPubTopic>
+        <control_channels>
+          <channel name="rotor4">
+            <input_index>4</input_index>
+            <input_offset>0</input_offset>
+            <input_scaling>3500</input_scaling>
+            <zero_position_disarmed>0</zero_position_disarmed>
+            <zero_position_armed>0</zero_position_armed>
+            <joint_control_type>velocity</joint_control_type>
+            <joint_name>rotor_puller_joint</joint_name>
+          </channel>
+          <channel name="left_elevon">
+            <input_index>5</input_index>
+            <input_offset>0</input_offset>
+            <input_scaling>1</input_scaling>
+            <zero_position_disarmed>0</zero_position_disarmed>
+            <zero_position_armed>0</zero_position_armed>
+            <joint_control_type>position_kinematic</joint_control_type>
+            <joint_name>left_elevon_joint</joint_name>
+          </channel>
+          <channel name="right_elevon">
+            <input_index>6</input_index>
+            <input_offset>0</input_offset>
+            <input_scaling>1</input_scaling>
+            <zero_position_disarmed>0</zero_position_disarmed>
+            <zero_position_armed>0</zero_position_armed>
+            <joint_control_type>position_kinematic</joint_control_type>
+            <joint_name>right_elevon_joint</joint_name>
+          </channel>
+          <channel name="elevator">
+            <input_index>7</input_index>
+            <input_offset>0</input_offset>
+            <input_scaling>1</input_scaling>
+            <zero_position_disarmed>0</zero_position_disarmed>
+            <zero_position_armed>0</zero_position_armed>
+            <joint_control_type>position_kinematic</joint_control_type>
+            <joint_name>elevator_joint</joint_name>
           </channel>
         </control_channels>

File: models/rotors_description/urdf/fixedwing_base.xacro (robot description, xacro)
@@ -21,107 +21,4 @@
          </collision>
       </link>
-      <!-- ELEVATORS-->
-      <!-- <link name="elevator">
-         <inertial>
-            <mass value="0.00001" />
-            <inertia ixx="0.00381666666667" ixy="0.0" ixz="0.0" iyy="0.0036" iyz="0.0" izz="0.00381666666667" />
-            <origin xyz="0 0 0" rpy="0 0 0" />
-         </inertial>
-         <collision name="collision">
-            <geometry>
-               <mesh filename="package://ardupilot_sitl_gazebo_plugin/meshes/meshes_drones/cessna/elevators.dae" />
-            </geometry>
-            <origin xyz="5.55 0 -0.57" rpy="0 0 0" />
-         </collision>
-         <visual name="visual">
-            <geometry>
-               <mesh filename="package://ardupilot_sitl_gazebo_plugin/meshes/meshes_drones/cessna/elevators.dae" />
-            </geometry>
-            <origin xyz="5.55 0 -0.57" rpy="0 0 0" />
-         </visual>
-      </link> -->
-      <!-- ELEVATORS JOINT-->
-      <!-- <joint name="elevator_joint" type="revolute">
-         <parent link="body" />
-         <child link="elevator" />
-         <origin xyz="-5.55 0 0.57" rpy="0 0 0" />
-         <axis xyz="0 1 0" />
-         <limit effort="-1" lower="-0.53" upper="0.53" velocity="-1" />
-         <dynamics damping="1.000" />
-      </joint> -->
-      <!-- RUDDER-->
-      <!-- <link name="rudder">
-         <inertial>
-            <mass value="0.00001" />
-            <inertia ixx="0.00381666666667" ixy="0.0" ixz="0.0" iyy="0.0036" iyz="0.0" izz="0.00381666666667" />
-            <origin xyz="-0.2 0 0" rpy="0 0 0" />
-         </inertial>
-         <collision name="collision">
-            <geometry>
-               <mesh filename="package://ardupilot_sitl_gazebo_plugin/meshes/meshes_drones/cessna/rudder.dae" />
-            </geometry>
-            <origin xyz="5.1 0 -3.25" rpy="0 0.35 0" />
-         </collision>
-         <visual name="visual">
-            <geometry>
-               <mesh filename="package://ardupilot_sitl_gazebo_plugin/meshes/meshes_drones/cessna/rudder.dae" />
-            </geometry>
-            <origin xyz="5.1 0 -3.25" rpy="0 0.35 0" />
-         </visual>
-      </link> -->
-      <!-- RUDDER JOINT-->
-      <!-- <joint name="rudder_joint" type="revolute">
-         <parent link="body" />
-         <child link="rudder" />
-         <origin xyz="-5.9 0 1.3" rpy="0 -0.35 0" />
-         <axis xyz="0 0 1" />
-         <limit effort="-1" lower="-0.53" upper="0.53" velocity="-1" />
-         <dynamics damping="1.000" />
-      </joint> -->
-      <!-- PROPELLER-->
-      <!-- <link name="rotor_puller">
-         <inertial>
-            <mass value="0.005" />
-            <inertia ixx="9.75e-07" ixy="0.00" iyy="0.000166704" ixz="0.00" iyz="0.00" izz="0.000167604" />
-            <origin xyz="0.3 0 0.0" rpy="0 1.57 0" />
-         </inertial>
-         <collision name="collision">
-            <geometry>
-               <cylinder length="0.005" radius="0.1"/>
-            </geometry>
-         </collision>
-         <visual name="visual">
-            <geometry>
-               <uri>model://rotors_description/meshes/iris_prop_ccw.dae</uri>
-            </geometry>
-         </visual>
-      </link> -->
-      <!-- PROPELLER JOINT-->
-      <!-- <joint name="rotor_puller_joint" type="revolute">
-         <parent link="body" />
-         <child link="propeller" />
-         <origin xyz="1.79 0 0.855" rpy="0 0 0" />
-         <axis xyz="1 0 0" />
-         <limit effort="-1" lower="-1e+16" upper="1e+16" velocity="-1" />
-           <dynamics damping="0.001" />
-      </joint> -->
-      <!-- <gazebo reference="right_aileron_joint">
-         <implicitSpringDamper>1</implicitSpringDamper>
-      </gazebo>
-      <gazebo reference="left_aileron_joint">
-         <implicitSpringDamper>1</implicitSpringDamper>
-      </gazebo>
-      <gazebo reference="left_flap_joint">
-         <implicitSpringDamper>1</implicitSpringDamper>
-      </gazebo>
-      <gazebo reference="right_flap_joint">
-         <implicitSpringDamper>1</implicitSpringDamper>
-      </gazebo>
-      <gazebo reference="rudder_joint">
-         <implicitSpringDamper>1</implicitSpringDamper>
-      </gazebo>
-      <gazebo reference="elevator_joint">
-         <implicitSpringDamper>1</implicitSpringDamper>
-      </gazebo> -->
       <gazebo>
          <link name='rotor_puller'>

File: models/rotors_description/urdf/plane_base.xacro (robot description, xacro)
@@ -70,5 +70,5 @@
   <xacro:if value="$(arg enable_mavlink_interface)">
   <!-- Instantiate mavlink telemetry interface. -->
-  <xacro:mavlink_interface_macro
+  <xacro:mavlink_interface_macro_fw
     namespace="${namespace}"
     imu_sub_topic="/imu"
@@ -94,5 +94,5 @@
     use_tcp="$(arg use_tcp)"
     >
-  </xacro:mavlink_interface_macro>
+  </xacro:mavlink_interface_macro_fw>
   </xacro:if>
   <!-- Mount an ADIS16448 IMU. -->
